Commit message: {playground_builder->freeplay_sandbox}

File: urdf/face_0.urdf (robot description, URDF)
Before this commit: robot face_0, 1 links, 0 joints
Links:
- link face_0: geometry visual mesh filename=package://freeplay_sandbox/meshes/child-face.dae

File: urdf/face_1.urdf (robot description, URDF)
Before this commit: robot face_1, 1 links, 0 joints
Links:
- link face_1: geometry visual mesh filename=package://freeplay_sandbox/meshes/child-face.dae

File: urdf/sandtray.urdf (robot description, URDF)
Before this commit: robot sandtray, 3 links, 2 joints
Links:
- link sandtray: geometry visual mesh filename=package://freeplay_sandbox/meshes/sandtray.dae
