Commit message: [sandtray urdf] Fixed orientation of camera base frames

File: urdf/sandtray.urdf (robot description, URDF)
Before this commit: robot sandtray, 3 links, 2 joints
Joints:
- joint l_camera_joint: origin xyz=-0.134 -0.004 0.019 rpy=0 -1.86 0.78 -> xyz=-0.134 -0.004 0.019 rpy=0 -0.292 0.785
- joint r_camera_joint: origin xyz=-0.134 0.346 0.019 rpy=0 -1.86 -0.78 -> xyz=-0.134 0.346 0.019 rpy=0 -0.292 -0.785

Commit message: Hopefully final URDF/DAE model of the sandtray

File: urdf/sandtray.urdf (robot description, URDF)
Before this commit: robot sandtray, 3 links, 2 joints
Joints:
- joint l_camera_joint: origin xyz=-0.134 -0.004 0.019 rpy=0 -0.292 0.785 -> xyz=-0.134 -0.351 0.025 rpy=0 -0.292 0.785
- joint r_camera_joint: origin xyz=-0.134 0.346 0.019 rpy=0 -0.292 -0.785 -> xyz=-0.134 -0.005 0.025 rpy=0 -0.292 -0.785

Commit message: Updated sandtray DAE/urdf for pilot study

File: urdf/sandtray.urdf (robot description, URDF)
Before this commit: robot sandtray, 3 links, 2 joints
Links:
- added link env_camera_link
Joints:
- added joint env_camera_joint: type fixed, parent sandtray, child env_camera_link, origin xyz=1.4 -0.15 0.52 rpy=0 0.29 3.142
- joint r_camera_joint: origin xyz=-0.134 -0.005 0.025 rpy=0 -0.292 -0.785 -> xyz=-0.006 -0.483 0.025 rpy=0 -0.326 1.347
