Commit message: Properly generate a sandtray.urdf with correct camera link names using xacro

File: urdf/sandtray.xacro (robot description, xacro)
@@ -7,24 +7,24 @@
     </visual>
   </link>
-  <link name="r_camera_link" />
-  <link name="l_camera_link" />
-  <link name="env_camera_link" />
+  <link name="$(arg camera1)_link" />
+  <link name="$(arg camera2)_link" />
+  <link name="$(arg env_camera)_link" />
     <!-- obtained from Blender: select frame in Blender, open Python console, then:
     >>> C.selected_objects[0].matrix_world.to_translation()
     >>> C.selected_objects[0].matrix_world.to_euler()
     -->
-  <joint name="r_camera_joint" type="fixed">
+  <joint name="$(arg camera1)_joint" type="fixed">
     <parent link="sandtray"/>
-    <child link="r_camera_link"/>
+    <child link="$(arg camera1)_link"/>
     <origin xyz="-0.006 -0.483 0.025" rpy="0 -0.326 1.347" />
   </joint>
-  <joint name="l_camera_joint" type="fixed">
+  <joint name="$(arg camera2)_joint" type="fixed">
     <parent link="sandtray"/>
-    <child link="l_camera_link"/>
+    <child link="$(arg camera2)_link"/>
     <origin xyz="-0.134 -0.351 0.025" rpy="0 -0.292 0.785" />
   </joint>
-  <joint name="env_camera_joint" type="fixed">
+  <joint name="$(arg env_camera)_joint" type="fixed">
     <parent link="sandtray"/>
-    <child link="env_camera_link"/>
+    <child link="$(arg env_camera)_link"/>
     <origin xyz="1.4 -0.15 0.52" rpy="0 0.29 3.142" />
   </joint>

Commit message: Updated sandtray model with SR300 v2 + new brackets

File: urdf/sandtray.xacro (robot description, xacro)
@@ -12,15 +12,15 @@
     <!-- obtained from Blender: select frame in Blender, open Python console, then:
     >>> C.selected_objects[0].matrix_world.to_translation()
-    >>> C.selected_objects[0].matrix_world.to_euler()
+    >>> C.selected_objects[0].matrix_world.to_euler() (making sure it is 'XYZ' eulers)
     -->
   <joint name="$(arg camera1)_joint" type="fixed">
     <parent link="sandtray"/>
     <child link="$(arg camera1)_link"/>
-    <origin xyz="-0.006 -0.483 0.025" rpy="0 -0.326 1.347" />
+    <origin xyz="-0.108 0.021 0.035" rpy="0 -0.349 -0.785" />
   </joint>
   <joint name="$(arg camera2)_joint" type="fixed">
     <parent link="sandtray"/>
     <child link="$(arg camera2)_link"/>
-    <origin xyz="-0.134 -0.351 0.025" rpy="0 -0.292 0.785" />
+    <origin xyz="-0.108 -0.377 0.035" rpy="0 -0.349 0.785" />
   </joint>
   <joint name="$(arg env_camera)_joint" type="fixed">
